File: Hardware/Wifi_WX_Station/as5040.brd (EAGLE design)
At the start: 25.4 x 25.3 mm, 16 parts

Commit message: backup
Parts:
- U$2: device 1AA_Stofer:TSSOP16 -> 1AA_Stofer:AMS_5040_SPECIAL
- moved C1 9.84 mm to (14.0, 18.7)
- moved U$2 3.88 mm to (10.8, 16.2)
- moved C5 1.62 mm to (14.0, 21.0)
Connections:
- net N$10: now also U$2.P$8; no longer U$2.8
- net N$11: now also U$2.P$12; no longer U$2.12
- net N$12: now also U$2.P$11; no longer U$2.11
- net N$13: now also U$2.P$10; no longer U$2.10
- net N$14: now also U$2.P$9; no longer U$2.9
- net N$2: now also U$2.P$7; no longer U$2.7
- net N$3: now also U$2.P$16; no longer U$2.16
- net N$4: now also U$2.P$15; no longer U$2.15
- net N$5: now also U$2.P$1; no longer U$2.1
- net N$6: now also U$2.P$2; no longer U$2.2
- net N$7: now also U$2.P$3; no longer U$2.3
- net N$8: now also U$2.P$4; no longer U$2.4
- net N$9: now also U$2.P$6; no longer U$2.6
Routing:
- net N$2: track 17.1 -> 28.8 mm, vias 0 -> 2
- net N$8: track 8.20 -> 7.31 mm
- net N$11: track 8.84 -> 7.95 mm
- net N$12: track 6.31 -> 5.42 mm
- net N$7: track 6.90 -> 6.01 mm
- net N$9: track 8.49 -> 7.60 mm
- net N$13: track 7.52 -> 6.63 mm
- net N$6: track 7.84 -> 6.95 mm
- net N$14: track 6.87 -> 5.98 mm
- net N$5: track 6.55 -> 5.78 mm
- net N$4: track 16.8 -> 16.1 mm, vias 0 -> 1
