File: Hardware/Wifi_WX_Station/as5040.sch (EAGLE design)
At the start: 16 parts

Commit message: backup
Changed lines of the file:
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@@
 <?xml version="1.0" encoding="utf-8"?>
 <!DOCTYPE eagle SYSTEM "eagle.dtd">
-<eagle version="6.3">
+<eagle version="6.5.0">
 <drawing>
 <settings>
