File: Hardware/Wifi_WX_Station/wind_speed.sch (EAGLE design)
At the start: 10 parts, among them T1 MMBT3904

Commit message: backup
Parts:
- OPTO1: value OSRAM_SHF9201 -> OSRAM_SFH9201
Changed lines of the file:
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@@
 <?xml version="1.0" encoding="utf-8"?>
 <!DOCTYPE eagle SYSTEM "eagle.dtd">
-<eagle version="6.3">
+<eagle version="6.5.0">
 <drawing>
 <settings>
@@
 </classes>
 <parts>
-<part name="OPTO1" library="wifi_WX" deviceset="OSRAM_SHF9201" device=""/>
+<part name="OPTO1" library="wifi_WX" deviceset="OSRAM_SHF9201" device="" value="OSRAM_SFH9201"/>
 <part name="T1" library="transistor" deviceset="BC846" device="" value="MMBT3904"/>
 <part name="R1" library="rcl" deviceset="R-US_" device="R0603" value="10K"/>
