File: Hardware/Wifi_WX_Station/Base.brd (EAGLE design)
At the start: 91.4 x 50.8 mm, 75 parts, among them IC1 3.3v, J1 RJ45-8VERT, J5 RJ11-6VERT_LP, J6 M05X22X5FE, Q1 32.768Khz, U1 CP2104-GM, U2 25LC512, U3 PIC24FJ128GA008

Commit message: added/changed some comments on schematic regarding Wind dir build options
Parts:
- R5: value 8.2k -> 14K
Changed lines of the file:
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@@
 <?xml version="1.0" encoding="utf-8"?>
 <!DOCTYPE eagle SYSTEM "eagle.dtd">
-<eagle version="6.3">
+<eagle version="6.4">
 <drawing>
 <settings>
@@
 <attribute name="NAME" x="13.6525" y="29.845" size="1.016" layer="25" rot="R270"/>
 </element>
-<element name="R5" library="rcl" package="R0603" value="8.2k" x="25.7175" y="24.4475" smashed="yes">
+<element name="R5" library="rcl" package="R0603" value="14K" x="25.7175" y="24.4475" smashed="yes">
 <attribute name="NAME" x="24.765" y="22.225" size="0.889" layer="25"/>
 </element>
