File: Hardware/Wifi_WX_Station/Base.sch (EAGLE design)
At the start: 75 parts, among them IC1 3.3v, J1 RJ45-8VERT, J5 RJ11-6VERT_LP, J6 M05X22X5FE, Q1 32.768Khz, U1 CP2104-GM, U2 25LC512, U3 PIC24FJ128GA008

Commit message: added/changed some comments on schematic regarding Wind dir build options
Parts:
- R5: value 8.2k -> 14K
Other:
- note added: "R6 - do not load for 3V WE28 Wind direction Sensor."
- note removed: "R6 - do not load for revision B.1 Wind Direction Sensor"
Changed lines of the file:
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@@
 <?xml version="1.0" encoding="utf-8"?>
 <!DOCTYPE eagle SYSTEM "eagle.dtd">
-<eagle version="6.3">
+<eagle version="6.4">
 <drawing>
 <settings>
@@
 <part name="C2" library="rcl" deviceset="C-US" device="C0805" value="0.1uF"/>
 <part name="P+1" library="supply1" deviceset="+5V" device=""/>
-<part name="R5" library="rcl" deviceset="R-US_" device="R0603" value="8.2k"/>
+<part name="R5" library="rcl" deviceset="R-US_" device="R0603" value="14K"/>
 <part name="R6" library="rcl" deviceset="R-US_" device="R0603" value="26.1K"/>
 <part name="C9" library="rcl" deviceset="C-US" device="C0805" value="0.1uF"/>
@@
 <text x="-83.82" y="55.88" size="1.27" layer="95">PIC24FJ256GA108</text>
 <text x="43.18" y="78.74" size="1.778" layer="95">MRF24</text>
-<text x="-226.06" y="-40.64" size="1.778" layer="96">R6 - do not load for revision B.1 Wind Direction Sensor</text>
+<text x="-226.06" y="-40.64" size="1.778" layer="96">R6 - do not load for 3V WE28 Wind direction Sensor. </text>
 <text x="118.872" y="-59.69" size="3.81" layer="94" ratio="15">B.2</text>
 <text x="35.56" y="-38.1" size="3.81" layer="94" ratio="15">WunderWxStation</text>
