File: Hardware/Wifi_WX_Station/RJ11_BoshBaro_SiHyg.brd (EAGLE design)
At the start: 24.8 x 20 mm, 8 parts, among them U1 SI7021-DFN6

Commit message: added/changed some comments on schematic regarding Wind dir build options
Parts:
- U2: value (none) -> BMP085
Changed lines of the file:
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@@
 <?xml version="1.0" encoding="utf-8"?>
 <!DOCTYPE eagle SYSTEM "eagle.dtd">
-<eagle version="6.5.0">
+<eagle version="6.4">
 <drawing>
 <settings>
@@
 <attribute name="NAME" x="26.43" y="4.715" size="1.016" layer="25" rot="R90"/>
 </element>
-<element name="U2" library="1AA_Stofer" package="LCC8" value="" x="15.875" y="5.08" smashed="yes" rot="R180"/>
+<element name="U2" library="1AA_Stofer" package="LCC8" value="BMP085" x="15.875" y="5.08" smashed="yes" rot="R180"/>
 <element name="JP2" library="wifi_WX" package="RJ11_HOR_LP" value="RJ11-6HOR_LP" x="29.845" y="9.525" rot="MR270"/>
 <element name="U1" library="wifi_WX" package="DFN-6_SILABS" value="SI7021-DFN6" x="12.3825" y="13.97" smashed="yes">
