File: Hardware/Wifi_WX_Station/RJ11_BoshBaro_SiHyg.sch (EAGLE design)
At the start: 8 parts, among them U1 SI7021-DFN6

Commit message: added/changed some comments on schematic regarding Wind dir build options
Parts:
- U2: value (none) -> BMP085
Changed lines of the file:
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@@
 <?xml version="1.0" encoding="utf-8"?>
 <!DOCTYPE eagle SYSTEM "eagle.dtd">
-<eagle version="6.5.0">
+<eagle version="6.4">
 <drawing>
 <settings>
@@
 <part name="C3" library="rcl" deviceset="CPOL-US" device="SMCB" value="22uF/10V"/>
 <part name="C1" library="rcl" deviceset="C-US" device="C0805K" value="100nF"/>
-<part name="U2" library="1AA_Stofer" deviceset="BMP085" device=""/>
+<part name="U2" library="1AA_Stofer" deviceset="BMP085" device="" value="BMP085"/>
 <part name="JP2" library="wifi_WX" deviceset="RJ11-6" device="HOR_LP"/>
 <part name="U$1" library="1AA_Stofer" deviceset="8.5X11" device=""/>
